Commit message: Make 6DOF

File: urdf/robot_arm.urdf.xacro (robot description, xacro)
@@ -16,4 +16,7 @@
   <material name="black">
     <color rgba="0.0 0.0 0.0 1.0"/>
+  </material>
+  <material name="orange">
+    <color rgba="1.0 0.5 0.0 1.0"/>
   </material>
   <!-- Base Link -->
@@ -118,14 +121,14 @@
     </inertial>
   </link>
-  <!-- Joint 4: Forearm to Wrist -->
+  <!-- Joint 4: Forearm to Wrist Roll -->
   <joint name="joint4" type="revolute">
     <parent link="forearm_link"/>
-    <child link="wrist_link"/>
+    <child link="wrist_roll_link"/>
     <origin xyz="0.25 0 0" rpy="0 0 0"/>
     <axis xyz="1 0 0"/>
     <limit lower="-1.57" upper="1.57" effort="50" velocity="1.0"/>
   </joint>
-  <!-- Wrist Link -->
-  <link name="wrist_link">
+  <!-- Wrist Roll Link -->
+  <link name="wrist_roll_link">
     <visual>
       <origin xyz="0.05 0 0" rpy="0 1.57 0"/>
@@ -146,9 +149,37 @@
     </inertial>
   </link>
-  <!-- Joint 5: Wrist Rotation -->
+  <!-- Joint 5: Wrist Roll to Wrist Pitch (NEW JOINT) -->
   <joint name="joint5" type="revolute">
-    <parent link="wrist_link"/>
+    <parent link="wrist_roll_link"/>
+    <child link="wrist_pitch_link"/>
+    <origin xyz="0.1 0 0" rpy="0 0 0"/>
+    <axis xyz="0 1 0"/>
+    <limit lower="-1.57" upper="1.57" effort="25" velocity="1.5"/>
+  </joint>
+  <!-- Wrist Pitch Link (NEW LINK) -->
+  <link name="wrist_pitch_link">
+    <visual>
+      <origin xyz="0.04 0 0" rpy="0 0 0"/>
+      <geometry>
+        <cylinder radius="0.02" length="0.08"/>
+      </geometry>
+      <material name="orange"/>
+    </visual>
+    <collision>
+      <origin xyz="0.04 0 0" rpy="0 0 0"/>
+      <geometry>
+        <cylinder radius="0.02" length="0.08"/>
+      </geometry>
+    </collision>
+    <inertial>
+      <mass value="0.15"/>
+      <inertia ixx="0.001" ixy="0.0" ixz="0.0" iyy="0.001" iyz="0.0" izz="0.001"/>
+    </inertial>
+  </link>
+  <!-- Joint 6: Wrist Pitch to Hand (previously joint5) -->
+  <joint name="joint6" type="revolute">
+    <parent link="wrist_pitch_link"/>
     <child link="hand_link"/>
-    <origin xyz="0.1 0 0" rpy="0 0 0"/>
+    <origin xyz="0.08 0 0" rpy="0 0 0"/>
     <axis xyz="0 0 1"/>
     <limit lower="-3.14" upper="3.14" effort="25" velocity="1.5"/>
@@ -236,5 +267,5 @@
     <parent link="base_link"/>
     <child link="shoulder_link_second_arm"/>
-    <origin xyz="0 0 0.1" rpy="0 0 3.14"/>
+    <origin xyz="1 0 0.1" rpy="0 0 3.14"/>
     <axis xyz="0 0 1"/>
     <limit lower="-3.14" upper="3.14" effort="100" velocity="1.0"/>
@@ -314,14 +345,14 @@
     </inertial>
   </link>
-  <!-- Joint 4: Forearm to Wrist -->
+  <!-- Joint 4: Forearm to Wrist Roll -->
   <joint name="joint4_second_arm" type="revolute">
     <parent link="forearm_link_second_arm"/>
-    <child link="wrist_link_second_arm"/>
+    <child link="wrist_roll_link_second_arm"/>
     <origin xyz="0.25 0 0" rpy="0 0 0"/>
     <axis xyz="1 0 0"/>
     <limit lower="-1.57" upper="1.57" effort="50" velocity="1.0"/>
   </joint>
-  <!-- Wrist Link -->
-  <link name="wrist_link_second_arm">
+  <!-- Wrist Roll Link -->
+  <link name="wrist_roll_link_second_arm">
     <visual>
       <origin xyz="0.05 0 0" rpy="0 1.57 0"/>
@@ -342,9 +373,37 @@
     </inertial>
   </link>
-  <!-- Joint 5: Wrist Rotation -->
+  <!-- Joint 5: Wrist Roll to Wrist Pitch (NEW JOINT) -->
   <joint name="joint5_second_arm" type="revolute">
-    <parent link="wrist_link_second_arm"/>
+    <parent link="wrist_roll_link_second_arm"/>
+    <child link="wrist_pitch_link_second_arm"/>
+    <origin xyz="0.1 0 0" rpy="0 0 0"/>
+    <axis xyz="0 1 0"/>
+    <limit lower="-1.57" upper="1.57" effort="25" velocity="1.5"/>
+  </joint>
+  <!-- Wrist Pitch Link (NEW LINK) -->
+  <link name="wrist_pitch_link_second_arm">
+    <visual>
+      <origin xyz="0.04 0 0" rpy="0 0 0"/>
+      <geometry>
+        <cylinder radius="0.02" length="0.08"/>
+      </geometry>
+      <material name="orange"/>
+    </visual>
+    <collision>
+      <origin xyz="0.04 0 0" rpy="0 0 0"/>
+      <geometry>
+        <cylinder radius="0.02" length="0.08"/>
+      </geometry>
+    </collision>
+    <inertial>
+      <mass value="0.15"/>
+      <inertia ixx="0.001" ixy="0.0" ixz="0.0" iyy="0.001" iyz="0.0" izz="0.001"/>
+    </inertial>
+  </link>
+  <!-- Joint 6: Wrist Pitch to Hand (previously joint5) -->
+  <joint name="joint6_second_arm" type="revolute">
+    <parent link="wrist_pitch_link_second_arm"/>
     <child link="hand_link_second_arm"/>
-    <origin xyz="0.1 0 0" rpy="0 0 0"/>
+    <origin xyz="0.08 0 0" rpy="0 0 0"/>
     <axis xyz="0 0 1"/>
     <limit lower="-3.14" upper="3.14" effort="25" velocity="1.5"/>
